File: Electronics/Circuit Monitor.sch (KiCad schematic (older format))
At the start: 31 parts

Commit message: More schematic progress and removed diagrams to fix bug
Parts:
- added Q? (x4): HCPL-181-00DE, SOIC254P700X220-4N, symbol HCPL-181-00DE
- added R? (x4): 100R, symbol R_Small
- added R? (x8): 1K, symbol R_Small
Connections:
- net +3V3: now also U?.1 (Vdd1), R?.2, R?.2, R?.2, R?.2; no longer R?.1
- net GNDA: now also U?.5 (GND2)
- net GNDD: now also Q?.2 (C), Q?.2 (C), Q?.2 (C), Q?.2 (C)
- net TX: now reaches U?.12 (UART_TX)
- net TX: now also R?.1
- net RX: now reaches U?.5 (COMMONa)
- net RX: now also R?.1
- net at U?.2 (Voa): now also R?.1
- net at U?.3 (Vinb): now also R?.1
- net GND: now reaches U?.4 (GND1)
- net GND: now also Q?.3 (ET), Q?.3 (ET), Q?.3 (ET), Q?.3 (ET)
- net at U?.6 (Vob): now also R?.2
- net at U?.7 (Vina): now also R?.2
- net +3.3VP: now reaches U?.8 (Vdd2)
- net +3.3VP: now also R?.1
- new net: Q?.1 (A), R?.2 (x4)
- new net EVENT1: R?.1
- new net EVENT1I: Q?.4 (CT), R?.1
- new net EVENT2: R?.1
- new net EVENT2I: Q?.4 (CT), R?.1
- new net PWM: R?.1
- new net PWMI: Q?.4 (CT), R?.1
- new net RXI: R?.2
- new net TXI: R?.2
- new net ZCD: R?.1
- new net ZCDI: Q?.4 (CT), R?.1
