File: Electronics/_saved_Circuit Monitor.sch (KiCad schematic (older format))
At the start: 37 parts

Commit message: More schematic progress and removed diagrams to fix bug
Parts:
- removed Q? (x3): HCPL-181-00DE, SOIC254P700X220-4N, symbol HCPL-181-00DE
- added Q? (x3): HCPL-181-00DE, SOIC254P700X220-4N, symbol HCPL-181-00DE
- added R? (x8): 1K, symbol R_Small
- added R? (x2): 100R, symbol R_Small
Connections:
- net GNDD: now also Q?.2 (C), Q?.2 (C), Q?.2 (C), Q?.2 (C)
- net at Q?.1 (A): now also R?.2
- net GND: now reaches Q?.3 (ET)
- net GND: now also U?.4 (GND1), Q?.3 (ET), Q?.3 (ET), Q?.3 (ET)
- net EVENT1I: now reaches Q?.4 (CT)
- net EVENT1I: now also R?.1
- net +3V3: now reaches U?.1 (Vdd1)
- net +3V3: now also R?.2, R?.2, R?.2, R?.2
- net at U?.2 (Voa): now also R?.1
- net at U?.3 (Vinb): now also R?.1
- new net: Q?.1 (A), R?.2 (x3)
- new net EVENT1: R?.1
- new net EVENT2: R?.1
- new net EVENT2I: Q?.4 (CT), R?.1
- new net PWM: R?.1
- new net PWMI: Q?.4 (CT), R?.1
- new net RXI: R?.2
- new net TXI: R?.2
- new net ZCD: R?.1
- new net ZCDI: Q?.4 (CT), R?.1
Other:
- moved on the sheet: Q?
